Commit message: rviz set

File: src/rover_description/urdf/rover.urdf.xacro (robot description, xacro)
@@ -2,6 +2,9 @@
 <robot xmlns:xacro="http://www.ros.org/wiki/xacro" name="rover">
     <xacro:arg name="use_sim" default="true"/>
-    <xacro:property name="chassis_length" value="0.24"/> <xacro:property name="chassis_width" value="0.18"/>  <xacro:property name="chassis_height" value="0.08"/>
-    <xacro:property name="wheel_radius" value="0.04"/>   <xacro:property name="wheel_width" value="0.04"/>
+    <xacro:property name="chassis_length" value="0.24"/>
+    <xacro:property name="chassis_width" value="0.18"/>
+    <xacro:property name="chassis_height" value="0.08"/>
+    <xacro:property name="wheel_radius" value="0.04"/>
+    <xacro:property name="wheel_width" value="0.04"/>
     <xacro:property name="wheel_offset_x" value="0.09"/>
     <xacro:property name="wheel_offset_y" value="0.10"/>
@@ -12,6 +15,6 @@
                 <box size="${chassis_length} ${chassis_width} ${chassis_height}"/>
             </geometry>
-            <material name="Silver">
-                <color rgba="0.75 0.75 0.75 1"/>
+            <material name="Blue">
+                <color rgba="0 0 1 1"/>
             </material>
             <origin xyz="0 0 ${chassis_height/2}"/>
@@ -67,5 +70,5 @@
             <parent link="base_link"/>
             <child link="${prefix}_wheel_link"/>
-            <origin xyz="${x_reflect * wheel_offset_x} ${y_reflect * wheel_offset_y} ${wheel_radius}" rpy="0 0 0"/>
+            <origin xyz="${x_reflect * wheel_offset_x} ${y_reflect * wheel_offset_y} 0" rpy="0 0 0"/>
             <axis xyz="0 1 0"/>
             <xacro:if value="${is_mimic}">

Commit message: refactoring

File: src/rover_description/urdf/rover.urdf.xacro (robot description, xacro)
@@ -31,4 +31,7 @@
         </inertial>
     </link>
+    <gazebo reference="base_link">
+        <material>Gazebo/Blue</material>
+    </gazebo>
     <joint name="base_joint" type="fixed">
         <parent link="base_footprint"/>
@@ -42,4 +45,7 @@
         </visual>
     </link>
+    <gazebo reference="laser_frame">
+        <material>Gazebo/Red</material>
+    </gazebo>
     <joint name="laser_joint" type="fixed">
         <parent link="base_link"/>
@@ -67,4 +73,9 @@
             </inertial>
         </link>
+        <gazebo reference="${prefix}_wheel_link">
+            <material>Gazebo/Black</material>
+            <mu1>1.0</mu1>
+            <mu2>1.0</mu2>
+        </gazebo>
         <joint name="${prefix}_wheel_joint" type="continuous">
             <parent link="base_link"/>
@@ -93,17 +104,23 @@
         </hardware>
         <joint name="rear_left_wheel_joint">
-            <command_interface name="velocity"><param name="min">-10</param><param name="max">10</param></command_interface>
+            <command_interface name="velocity">
+                <param name="min">-10</param>
+                <param name="max">10</param>
+            </command_interface>
             <state_interface name="velocity"/>
             <state_interface name="position"/>
         </joint>
         <joint name="rear_right_wheel_joint">
-            <command_interface name="velocity"><param name="min">-10</param><param name="max">10</param></command_interface>
+            <command_interface name="velocity">
+                <param name="min">-10</param>
+                <param name="max">10</param>
+            </command_interface>
             <state_interface name="velocity"/>
             <state_interface name="position"/>
         </joint>
     </ros2_control>
-    <gazebo>
+   <gazebo>
         <plugin name="gazebo_ros2_control" filename="libgazebo_ros2_control.so">
-            <parameters>$(find rover_bringup)/config/control.yaml</parameters>
+            <parameters>$(find rover_control)/config/control.yaml</parameters>
         </plugin>
     </gazebo>
